File: PCB/openDSO.sch (KiCad schematic (older format))
At the start: 1 part, among them J1 Z_TURN_Lite

Commit message: fix Zturn footprint
Parts:
- added U1: MAX19506, Housings_QFP:TQFP-48-1EP_7x7mm_Pitch0.5mm, symbol MAX19506
Changed lines of the file:
@@
 EESchema Schematic File Version 2
 LIBS:z_turn_lite
+LIBS:max19506
+LIBS:openDSO-cache
 EELAYER 26 0
 EELAYER END
@@
 	1    0    0    -1
 $EndComp
+$Comp
+L MAX19506 U1
+U 1 1 5CAF81E8
+P 6500 2700
+F 0 "U1" H 7050 1114 50  0000 C CNN
+F 1 "MAX19506" H 7050 1023 50  0000 C CNN
+F 2 "Housings_QFP:TQFP-48-1EP_7x7mm_Pitch0.5mm" H 6550 4150 50  0001 C CNN
+F 3 "" H 6450 2850 50  0001 C CNN
+	1    6500 2700
+	1    0    0    -1
+$EndComp
